Commit message: lower friction caster wheel

File: src/robot_vacuum_description/urdf/gazebo/gazebo_plugins.xacro (robot description, xacro)
@@ -21,6 +21,6 @@
             <joint_name>left_wheel_joint</joint_name>
             <joint_name>right_wheel_joint</joint_name>
-            <joint_name>caster_frame_joint</joint_name>
-            <joint_name>caster_wheel_joint</joint_name>
+            <!-- <joint_name>caster_frame_joint</joint_name> -->
+            <!--<joint_name>caster_wheel_joint</joint_name> -->
         </plugin>
     </gazebo>

File: src/robot_vacuum_description/urdf/gazebo/gazebo_properties.xacro (robot description, xacro)
@@ -38,12 +38,12 @@
   <!-- Caster Wheels -->
   <gazebo reference="caster_wheel_link">
-    <mu1 value="0.8"/>
-    <mu2 value="0.8"/>
-    <kp value="1000000.0"/>
-    <kd value="0.1"/>
-  </gazebo>
-  <gazebo reference="caster_frame_link">
     <mu1 value="0.1"/>
     <mu2 value="0.1"/>
+   <!--  <kp value="1000000.0"/>
+    <kd value="0.1"/> -->
   </gazebo>
+  <!-- <gazebo reference="caster_frame_link">
+    <mu1 value="0.05"/>
+    <mu2 value="0.05"/>
+  </gazebo> -->
 </robot>

File: src/robot_vacuum_description/urdf/modules/base_and_wheels.xacro (robot description, xacro)
@@ -180,18 +180,14 @@
   </link>
   <!-- Joint from caster_frame to caster_wheel -->
-  <joint name="caster_wheel_joint" type="continuous">
-    <origin xyz="-0.009 0.0145 -0.0192" rpy="-1.5708 -0 -0"/>
+  <joint name="caster_wheel_joint" type="fixed">
+    <origin xyz="-0.009 0.0145 -0.0192" rpy="-1.5708 0 0"/>
     <parent link="caster_frame_link"/>
     <child link="caster_wheel_link"/>
-    <axis xyz="0 0 1"/>
-    <limit effort="100" velocity="100"/>
   </joint>
   <!-- Joint from base_link to caster_frame -->
-  <joint name="caster_frame_joint" type="continuous">
+  <joint name="caster_frame_joint" type="fixed">
     <origin xyz="0.11 -0 0.014" rpy="0 -0 -3.14159"/>
     <parent link="base_link"/>
     <child link="caster_frame_link"/>
-    <axis xyz="0 0 1"/>
-    <limit effort="100" velocity="100"/>
   </joint>
 </robot>

Commit message: Revert "lower friction caster wheel"
This reverts commit 1abbd6a86c5a72dd409079b066056848796c7a74.

File: src/robot_vacuum_description/urdf/gazebo/gazebo_plugins.xacro (robot description, xacro)
@@ -21,6 +21,6 @@
             <joint_name>left_wheel_joint</joint_name>
             <joint_name>right_wheel_joint</joint_name>
-            <!-- <joint_name>caster_frame_joint</joint_name> -->
-            <!--<joint_name>caster_wheel_joint</joint_name> -->
+            <joint_name>caster_frame_joint</joint_name>
+            <joint_name>caster_wheel_joint</joint_name>
         </plugin>
     </gazebo>

File: src/robot_vacuum_description/urdf/gazebo/gazebo_properties.xacro (robot description, xacro)
@@ -38,12 +38,12 @@
   <!-- Caster Wheels -->
   <gazebo reference="caster_wheel_link">
+    <mu1 value="0.8"/>
+    <mu2 value="0.8"/>
+    <kp value="1000000.0"/>
+    <kd value="0.1"/>
+  </gazebo>
+  <gazebo reference="caster_frame_link">
     <mu1 value="0.1"/>
     <mu2 value="0.1"/>
-   <!--  <kp value="1000000.0"/>
-    <kd value="0.1"/> -->
   </gazebo>
-  <!-- <gazebo reference="caster_frame_link">
-    <mu1 value="0.05"/>
-    <mu2 value="0.05"/>
-  </gazebo> -->
 </robot>

File: src/robot_vacuum_description/urdf/modules/base_and_wheels.xacro (robot description, xacro)
@@ -180,14 +180,18 @@
   </link>
   <!-- Joint from caster_frame to caster_wheel -->
-  <joint name="caster_wheel_joint" type="fixed">
-    <origin xyz="-0.009 0.0145 -0.0192" rpy="-1.5708 0 0"/>
+  <joint name="caster_wheel_joint" type="continuous">
+    <origin xyz="-0.009 0.0145 -0.0192" rpy="-1.5708 -0 -0"/>
     <parent link="caster_frame_link"/>
     <child link="caster_wheel_link"/>
+    <axis xyz="0 0 1"/>
+    <limit effort="100" velocity="100"/>
   </joint>
   <!-- Joint from base_link to caster_frame -->
-  <joint name="caster_frame_joint" type="fixed">
+  <joint name="caster_frame_joint" type="continuous">
     <origin xyz="0.11 -0 0.014" rpy="0 -0 -3.14159"/>
     <parent link="base_link"/>
     <child link="caster_frame_link"/>
+    <axis xyz="0 0 1"/>
+    <limit effort="100" velocity="100"/>
   </joint>
 </robot>
