Commit message: fix lidar bug

File: src/robot_description/urdf/gazebo/gazebo_plugins.xacro (robot description, xacro)
@@ -9,6 +9,7 @@
             <wheel_separation>0.186</wheel_separation>
             <wheel_radius>0.0375</wheel_radius>
-            <frame_id>${robot_name}/odom</frame_id> <!--Best to use prefixes and to set the prefix on the RVIZ config too, see xacro_properties.xacro for where to change these -->
-            <child_frame_id>${robot_name}/base_footprint</child_frame_id>  <!--Best to use prefixes and to set the prefix on the RVIZ config too, see xacro_properties.xacro for where to change these -->
+            <frame_id>${robot_name}/odom</frame_id>
+            <child_frame_id>${robot_name}/base_footprint</child_frame_id>
+            <tf_topic>/model/${robot_name}/tf</tf_topic>
         </plugin>
     </gazebo>

File: src/robot_description/urdf/models/base_and_wheels.xacro (robot description, xacro)
@@ -3,7 +3,7 @@
 <!-- Onshape document_id: 6ec665232e6fc828980877e8 -->
 <robot name="robot_vacuum" xmlns:xacro="http://www.ros.org/wiki/xacro">
-  <link name="base_footprint_link"/>
+  <link name="base_footprint"/>
   <joint name="base_joint" type="fixed">
-    <parent link="base_footprint_link" />
+    <parent link="base_footprint" />
     <child link="base_link" />
     <origin xyz="0 0 0.025" rpy="0 0 0" />

File: src/robot_description/urdf/models/lidar.xacro (robot description, xacro)
@@ -14,5 +14,5 @@
       <origin xyz="0 0 0" rpy="0 0 0"/>
       <geometry>
-        <cylinder radius="0.03" length="0.01" />
+        <cylinder radius="0.03" length="0.015" />
       </geometry>
       <material name="lidar_link_material">
